File: PCB/Annelise/Annelise.kicad_pcb (KiCad board)
At the start: 2 copper layers, 278.6 x 86.7 mm, 87 parts, among them J1 Conn_01x04_Female, J2 Conn_01x03_Female, SW1 SW_Push_45deg, SW10 SW_Push_45deg, SW11 SW_Push_45deg, SW12 SW_Push_45deg, SW13 SW_Push_45deg, SW14 SW_Push_45deg, SW15 SW_Push_45deg, SW16 SW_Push_45deg, SW17 SW_Push_45deg, SW18 SW_Push_45deg, SW19 SW_Push_45deg, SW2 SW_Push_45deg, SW20 SW_Push_45deg, SW21 SW_Push_45deg, SW22 SW_Push_45deg, SW23 SW_Push_45deg, SW24 SW_Push_45deg, SW25 SW_Push_45deg, SW26 SW_Push_45deg, SW27 SW_Push_45deg, SW28 SW_Push_45deg, SW29 SW_Push_45deg, SW3 SW_Push_45deg, SW30 SW_Push_45deg, SW31 SW_Push_45deg, SW32 SW_Push_45deg, SW33 SW_Push_45deg, SW34 SW_Push_45deg, SW35 SW_Push_45deg, SW36 SW_Push_45deg, SW37 SW_Push_45deg, SW38 SW_Push_45deg, SW39 SW_Push_45deg, SW4 SW_Push_45deg, SW40 SW_Push_45deg, SW41 SW_Push_45deg, SW42 SW_Push_45deg, SW43 SW_Push_45deg, SW44 SW_Push_45deg, SW45 SW_Push_45deg, SW46 SW_Push_45deg, SW5 SW_Push_45deg, SW6 SW_Push_45deg, SW7 SW_Push_45deg, SW8 SW_Push_45deg, SW9 SW_Push_45deg, U2 STM32F103CBTx, U3 XC6206P332MR, Y1 Resonator_Small

Commit message: pcb updates
Parts:
- moved C1 108.3 mm to (166.0, 134.3), turned to 135 degrees
- moved R4 97.8 mm to (170.4, 122.3), turned to 315 degrees
- moved C5 97.5 mm to (156.7, 129.0), turned to 315 degrees
- moved C4 96.4 mm to (167.0, 133.2), turned to 315 degrees
- moved Y1 95.4 mm to (168.9, 131.4), turned to 225 degrees
- moved U3 86.4 mm to (171.9, 113.0), turned to 90 degrees
- moved J2 83.5 mm to (165.4, 115.0), turned to 90 degrees
- moved C7 77.5 mm to (159.1, 118.8), turned to 225 degrees
- moved R3 71.8 mm to (158.0, 117.7), turned to 225 degrees
- moved C6 66.2 mm to (160.2, 119.8), turned to 225 degrees
- moved C9 64.9 mm to (169.4, 113.0), turned to 90 degrees
- moved U2 62.2 mm to (163.0, 126.2), turned to 135 degrees
- moved C3 56.0 mm to (169.4, 123.4), turned to 135 degrees
- moved C8 45.4 mm to (174.4, 113.0)
- moved F1 43.7 mm to (168.1, 107.4)
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Connections:
- SW42 pad 2: Net-(SW42-Pad2) -> Net-(D21-Pad2)
- SW44 pad 2: Net-(SW44-Pad2) -> Net-(D22-Pad2)
- U2 pad 13: Net-(U2-Pad13) -> Row3
- U2 pad 14: Net-(U2-Pad14) -> Row2
- U2 pad 15: Net-(U2-Pad15) -> Row1
- U2 pad 16: Net-(U2-Pad16) -> Row0
- U2 pad 25: Net-(U2-Pad25) -> Col5
- U2 pad 26: Net-(U2-Pad26) -> Col4
- U2 pad 27: Net-(U2-Pad27) -> Col3
- U2 pad 28: Net-(U2-Pad28) -> Col2
- U2 pad 29: Net-(U2-Pad29) -> Col1
- U2 pad 30: Net-(U2-Pad30) -> Col0
- U2 pad 38: Net-(U2-Pad38) -> Col12
- U2 pad 39: Net-(U2-Pad39) -> Col11
- U2 pad 40: Net-(U2-Pad40) -> Col10
- U2 pad 41: Net-(U2-Pad41) -> Col9
- U2 pad 42: Net-(U2-Pad42) -> Col8
- U2 pad 43: Net-(U2-Pad43) -> Col7
- U2 pad 45: Net-(U2-Pad45) -> Col6
Routing:
- net Row0: track 0.00 -> 320.3 mm, vias 0 -> 2
- net Row1: track 0.00 -> 262.1 mm, vias 0 -> 2
- net Row3: track 0.00 -> 251.3 mm, vias 0 -> 2
- net Row2: track 0.00 -> 217.7 mm, vias 0 -> 2
- net Col12: track 0.00 -> 200.4 mm, vias 0 -> 1
- net Col11: track 0.00 -> 190.8 mm, vias 0 -> 1
- net Col0: track 0.00 -> 186.8 mm, vias 0 -> 1
- net Col1: track 0.00 -> 167.9 mm, vias 0 -> 1
- net Col10: track 0.00 -> 143.4 mm, vias 0 -> 1
- net Col2: track 0.00 -> 127.6 mm, vias 0 -> 1
- net Col3: track 0.00 -> 124.4 mm, vias 0 -> 1
- net Col9: track 0.00 -> 123.0 mm, vias 0 -> 1
- net Col8: track 0.00 -> 121.0 mm, vias 0 -> 1
- net Col4: track 0.00 -> 109.4 mm, vias 0 -> 2
- net Col7: track 0.00 -> 105.2 mm, vias 0 -> 1
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- added copper zone on B.Cu, net GND
- added copper zone on F.Cu, net GND

Commit message: pcb updates
Parts:
- removed R4: 10k, Resistor_SMD:R_0603_1608Metric
- added BOOT: SW_Push, Connector_PinHeader_1.27mm:PinHeader_1x02_P1.27mm_Vertical, B.Cu at (170.6, 136.3)
- added C2: 10uF, Capacitor_SMD:C_0603_1608Metric, B.Cu at (165.4, 136.4)
- added D24: BAT54C, Package_TO_SOT_SMD:SOT-23, B.Cu at (165.0, 139.4)
- added G***: LOGO, adela:exorcism, B.Cu at (160.8, 131.6)
- added Q1: DTC123J, Package_TO_SOT_SMD:SOT-23, B.Cu at (161.7, 139.4)
- added R1: 33k, Resistor_SMD:R_0603_1608Metric, B.Cu at (162.7, 136.4)
- added R2: 100k, Resistor_SMD:R_0603_1608Metric, B.Cu at (164.0, 136.4)
- C1: value 100nF -> 4.7uF
- moved C1 5.08 mm to (161.3, 136.4), turned to 270 degrees
- renumbered J2 to SWD
Connections:
- net Net-(C1-Pad2) renamed /RST
- U2 pad 44: Net-(R4-Pad1) -> /BOOT
Routing:
- net /BOOT: track 0.00 -> 21.3 mm, vias 0 -> 2
- net Net-(D24-Pad1): track 0.00 -> 10.7 mm, vias 0 -> 1
- net Net-(R4-Pad1): track 8.99 -> 0.00 mm, vias 2 -> 0
- net +3V3: track 66.2 -> 74.1 mm
- net Net-(D24-Pad3): track 0.00 -> 6.97 mm
- net /RST: track 9.79 -> 15.7 mm
- net GND: track 46.0 -> 51.5 mm
- net Row2: track 217.7 -> 220.3 mm
- net Row0: track 320.3 -> 320.9 mm
- net Col4: vias 2 -> 1
Other:
- board text added: "Annelise rev0.1 by @MarvFPV"
- board text added: "CLK"
- board text added: "GND"
- board text added: "IO"
