File: PCB/Annelise/Annelise.sch (KiCad schematic (older format))
At the start: 87 parts, among them J1 Conn_01x04_Female, J2 Conn_01x03_Female, SW1 SW_Push_45deg, SW10 SW_Push_45deg, SW11 SW_Push_45deg, SW12 SW_Push_45deg, SW13 SW_Push_45deg, SW14 SW_Push_45deg, SW15 SW_Push_45deg, SW16 SW_Push_45deg, SW17 SW_Push_45deg, SW18 SW_Push_45deg, SW19 SW_Push_45deg, SW2 SW_Push_45deg, SW20 SW_Push_45deg, SW21 SW_Push_45deg, SW22 SW_Push_45deg, SW23 SW_Push_45deg, SW24 SW_Push_45deg, SW25 SW_Push_45deg, SW26 SW_Push_45deg, SW27 SW_Push_45deg, SW28 SW_Push_45deg, SW29 SW_Push_45deg, SW3 SW_Push_45deg, SW30 SW_Push_45deg, SW31 SW_Push_45deg, SW32 SW_Push_45deg, SW33 SW_Push_45deg, SW34 SW_Push_45deg, SW35 SW_Push_45deg, SW36 SW_Push_45deg, SW37 SW_Push_45deg, SW38 SW_Push_45deg, SW39 SW_Push_45deg, SW4 SW_Push_45deg, SW40 SW_Push_45deg, SW41 SW_Push_45deg, SW42 SW_Push_45deg, SW43 SW_Push_45deg, SW44 SW_Push_45deg, SW45 SW_Push_45deg, SW46 SW_Push_45deg, SW5 SW_Push_45deg, SW6 SW_Push_45deg, SW7 SW_Push_45deg, SW8 SW_Push_45deg, SW9 SW_Push_45deg, U2 STM32F103CBTx, U3 XC6206P332MR, Y1 Resonator_Small

Commit message: pcb updates
Connections:
- net Col0: now also U2.30 (PA9)
- net Col1: now also U2.29 (PA8)
- net Col10: now also U2.40 (PB4)
- net Col11: now also U2.39 (PB3)
- net Col12: now also U2.38 (PA15)
- net Col2: now also U2.28 (PB15)
- net Col3: now also U2.27 (PB14)
- net Col4: now also U2.26 (PB13)
- net Col5: now also U2.25 (PB12)
- net Col6: now also U2.45 (PB8)
- net Col7: now also U2.43 (PB7)
- net Col8: now also U2.42 (PB6)
- net Col9: now also U2.41 (PB5)
- net Row0: now also U2.16 (PA6)
- net Row1: now also U2.15 (PA5)
- net Row2: now also U2.14 (PA4)
- net Row3: now also U2.13 (PA3)
- net at SW42.2: now also D21.2
- net at SW44.2: now also D22.2
Changed lines of the file:
@@
 	1    0    0    -1
 $EndComp
+Wire Wire Line
+	3800 3000 3850 3000
+Wire Wire Line
+	6950 3000 7000 3000
+Text GLabel 3000 6200 2    50   Input ~ 0
+Row0
+Text GLabel 3000 6100 2    50   Input ~ 0
+Row1
+Text GLabel 3000 6000 2    50   Input ~ 0
+Row2
+Text GLabel 3000 5900 2    50   Input ~ 0
+Row3
+Text GLabel 3000 6500 2    50   Input ~ 0
+Col0
+Text GLabel 3000 6400 2    50   Input ~ 0
+Col1
+Text GLabel 1700 7100 0    50   Input ~ 0
+Col2
+Text GLabel 1700 7000 0    50   Input ~ 0
+Col3
+Text GLabel 1700 6900 0    50   Input ~ 0
+Col4
+Text GLabel 1700 6800 0    50   Input ~ 0
+Col5
+Text GLabel 1700 6400 0    50   Input ~ 0
+Col6
+Text GLabel 1700 6300 0    50   Input ~ 0
+Col7
+Text GLabel 1700 6200 0    50   Input ~ 0
+Col8
+Text GLabel 1700 6100 0    50   Input ~ 0
+Col9
+Text GLabel 1700 6000 0    50   Input ~ 0
+Col10
+Text GLabel 1700 5900 0    50   Input ~ 0
+Col11
+Text GLabel 3000 7100 2    50   Input ~ 0
+Col12
 $EndSCHEMATC

Commit message: pcb updates
Parts:
- removed R4: 10k, Resistor_SMD:R_0603_1608Metric, symbol Device:R_Small
- added C2: 10uF, Capacitor_SMD:C_0603_1608Metric, symbol Device:C_Small
- added D24: BAT54C, Package_TO_SOT_SMD:SOT-23, symbol Diode:BAT54C
- added Q1: DTC123J, Package_TO_SOT_SMD:SOT-23, symbol Transistor_BJT:DTC123J
- added R1: 33k, Resistor_SMD:R_0603_1608Metric, symbol Device:R_Small
- added R2: 100k, Resistor_SMD:R_0603_1608Metric, symbol Device:R_Small
- added SW47: SW_Push, Connector_PinHeader_1.27mm:PinHeader_1x02_P1.27mm_Vertical, symbol Switch:SW_Push
- C1: value 100nF -> 4.7uF
Connections:
- net +3V3: now also SW47.2
- net GND: now also C2.2, Q1.2 (E), R2.1
- net BOOT: now reaches U2.44 (BOOT0)
- net BOOT: now also C2.1, R1.2, R2.2
- net RST: now reaches C1.2, U2.7 (NRST)
- net RST: now also Q1.3 (C)
- new net: D24.1, Q1.1 (B), SW47.1
- new net: D24.3, R1.1
- no-connect marks 0 -> 1
Changed lines of the file:
@@
 	1050 7450 950  7450
-$Comp
-L Device:R_Small R4
-U 1 1 60858195
-P 1000 4350
-F 0 "R4" V 1100 4350 50  0000 C CNN
-F 1 "10k" V 1150 4350 50  0000 C CNN
-F 2 "Resistor_SMD:R_0603_1608Metric" H 1000 4350 50  0001 C CNN
-F 3 "~" H 1000 4350 50  0001 C CNN
-	1    1000 4350
-	0    1    1    0
-$EndComp
-$Comp
-L Device:C_Small C1
-U 1 1 60859A76
-P 1000 4200
-F 0 "C1" V 1150 4200 50  0000 C CNN
-F 1 "100nF" V 1100 4200 50  0000 C CNN
-F 2 "Capacitor_SMD:C_0603_1608Metric" H 1000 4200 50  0001 C CNN
-F 3 "~" H 1000 4200 50  0001 C CNN
-	1    1000 4200
-	0    -1   -1   0
-$EndComp
-Wire Wire Line
-	1100 4350 1450 4350
-Wire Wire Line
-	1450 4350 1450 4700
-Wire Wire Line
-	1450 4700 1700 4700
-Wire Wire Line
-	1100 4200 1550 4200
-Wire Wire Line
-	1550 4200 1550 4500
-Wire Wire Line
-	1550 4500 1700 4500
-Wire Wire Line
-	900  4200 900  4350
-Wire Wire Line
-	900  4350 550  4350
-Wire Wire Line
-	550  4350 550  4950
-Wire Wire Line
-	550  4950 750  4950
-Connection ~ 900  4350
-Connection ~ 750  4950
 $Comp
 L Device:R_Small R3
@@
 Text GLabel 3000 7100 2    50   Input ~ 0
 Col12
+Text HLabel 1700 4500 0    50   Input ~ 0
+RST
+Text HLabel 1700 4700 0    50   Input ~ 0
+BOOT
+$Comp
+L Transistor_BJT:DTC123J Q1
+U 1 1 60B55D03
+P 9050 4700
+F 0 "Q1" V 9375 4700 50  0000 C CNN
+F 1 "DTC123J" V 9284 4700 50  0000 C CNN
+F 2 "Package_TO_SOT_SMD:SOT-23" H 9050 4700 50  0001 L CNN
+F 3 "" H 9050 4700 50  0001 L CNN
+	1    9050 4700
+	0    -1   -1   0
+$EndComp
+$Comp
+L Device:C_Small C1
+U 1 1 60B57DA6
+P 8750 4750
+F 0 "C1" H 8842 4796 50  0000 L CNN
+F 1 "4.7uF" H 8842 4705 50  0000 L CNN
+F 2 "Capacitor_SMD:C_0603_1608Metric" H 8750 4750 50  0001 C CNN
+F 3 "~" H 8750 4750 50  0001 C CNN
+	1    8750 4750
+	-1   0    0    1
+$EndComp
+Wire Wire Line
+	8750 4650 8750 4600
+Wire Wire Line
+	8750 4600 8850 4600
+Wire Wire Line
+	8750 4600 8650 4600
+Connection ~ 8750 4600
+Text HLabel 8650 4600 0    50   Input ~ 0
+RST
+$Comp
+L power:GND #PWR0110
+U 1 1 60B6B62C
+P 8750 4850
+F 0 "#PWR0110" H 8750 4600 50  0001 C CNN
+F 1 "GND" H 8755 4677 50  0000 C CNN
+F 2 "" H 8750 4850 50  0001 C CNN
+F 3 "" H 8750 4850 50  0001 C CNN
+	1    8750 4850
+	1    0    0    -1
+$EndComp
+$Comp
+L power:GND #PWR0116
+U 1 1 60B6D2EB
+P 9350 4600
+F 0 "#PWR0116" H 9350 4350 50  0001 C CNN
+F 1 "GND" H 9355 4427 50  0000 C CNN
+F 2 "" H 9350 4600 50  0001 C CNN
+F 3 "" H 9350 4600 50  0001 C CNN
+	1    9350 4600
+	1    0    0    -1
+$EndComp
+Wire Wire Line
+	9250 4600 9350 4600
+$Comp
+L Switch:SW_Push SW47
+U 1 1 60B72C31
+P 9400 5150
+F 0 "SW47" H 9400 5435 50  0000 C CNN
+F 1 "SW_Push" H 9400 5344 50  0000 C CNN
+F 2 "Connector_PinHeader_1.27mm:PinHeader_1x02_P1.27mm_Vertical" H 9400 5350 50  0001 C CNN
+F 3 "~" H 9400 5350 50  0001 C CNN
+	1    9400 5150
+	1    0    0    -1
+$EndComp
+Wire Wire Line
+	9050 4950 9050 5150
+Wire Wire Line
+	9050 5150 9200 5150
+Wire Wire Line
+	9600 5150 9650 5150
+Wire Wire Line
+	9650 5150 9650 5100
+$Comp
+L power:+3V3 #PWR0117
+U 1 1 60B7D972
+P 9650 5100
+F 0 "#PWR0117" H 9650 4950 50  0001 C CNN
+F 1 "+3V3" H 9665 5273 50  0000 C CNN
+F 2 "" H 9650 5100 50  0001 C CNN
+F 3 "" H 9650 5100 50  0001 C CNN
+	1    9650 5100
+	1    0    0    -1
+$EndComp
+$Comp
+L Diode:BAT54C D24
+U 1 1 60B7EDD9
+P 9050 5450
+F 0 "D24" V 9004 5538 50  0000 L CNN
+F 1 "BAT54C" V 9095 5538 50  0000 L CNN
+F 2 "Package_TO_SOT_SMD:SOT-23" H 9125 5575 50  0001 L CNN
+F 3 "http://www.diodes.com/_files/datasheets/ds11005.pdf" H 8970 5450 50  0001 C CNN
+	1    9050 5450
+	0    1    1    0
+$EndComp
+Connection ~ 9050 5150
+NoConn ~ 9050 5750
+$Comp
+L Device:R_Small R1
+U 1 1 60B89DD7
+P 8650 5450
+F 0 "R1" V 8454 5450 50  0000 C CNN
+F 1 "33k" V 8545 5450 50  0000 C CNN
+F 2 "Resistor_SMD:R_0603_1608Metric" H 8650 5450 50  0001 C CNN
+F 3 "~" H 8650 5450 50  0001 C CNN
+	1    8650 5450
+	0    1    1    0
+$EndComp
+Wire Wire Line
+	8750 5450 8850 5450
+$Comp
+L Device:R_Small R2
+U 1 1 60B8F42A
+P 8400 5600
+F 0 "R2" H 8341 5554 50  0000 R CNN
+F 1 "100k" H 8341 5645 50  0000 R CNN
+F 2 "Resistor_SMD:R_0603_1608Metric" H 8400 5600 50  0001 C CNN
+F 3 "~" H 8400 5600 50  0001 C CNN
+	1    8400 5600
+	-1   0    0    1
+$EndComp
+$Comp
+L Device:C_Small C2
+U 1 1 60B8F70E
+P 8050 5600
+F 0 "C2" H 8142 5646 50  0000 L CNN
+F 1 "10uF" H 8142 5555 50  0000 L CNN
+F 2 "Capacitor_SMD:C_0603_1608Metric" H 8050 5600 50  0001 C CNN
+F 3 "~" H 8050 5600 50  0001 C CNN
+	1    8050 5600
+	1    0    0    -1
+$EndComp
+Wire Wire Line
+	8050 5500 8050 5450
+Wire Wire Line
+	8400 5500 8400 5450
+Wire Wire Line
+	8050 5450 8400 5450
+Connection ~ 8400 5450
+Wire Wire Line
+	8400 5450 8550 5450
+Wire Wire Line
+	8400 5700 8250 5700
+$Comp
+L power:GND #PWR0118
+U 1 1 60BAB88F
+P 8250 5700
+F 0 "#PWR0118" H 8250 5450 50  0001 C CNN
+F 1 "GND" H 8255 5527 50  0000 C CNN
+F 2 "" H 8250 5700 50  0001 C CNN
+F 3 "" H 8250 5700 50  0001 C CNN
+	1    8250 5700
+	1    0    0    -1
+$EndComp
+Connection ~ 8250 5700
+Wire Wire Line
+	8250 5700 8050 5700
+Text HLabel 8050 5450 0    50   Input ~ 0
+BOOT
 $EndSCHEMATC
